File: flasher.kicad_sch (KiCad schematic)
At the start: 22 parts, among them Q2 SS8050_C2150, Q3 SS8050_C2150, U4 CH343G

Commit message: Updated
Parts:
- renumbered C6 to C10, C3 to C7, C4 to C8, C5 to C9, D6 to D10, D7 to D11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

Commit message: No idea why everything changed again. KiCAD is the most shitty software I have ever seen.
Parts:
- renumbered D10 to D6, D11 to D7, D12 to D8, D13 to D9, U10 to U5
